File: KicadFiles/bldc_controller_v2.sch (KiCad schematic (older format))
At the start: 162 parts, among them J1 Conn_01x06_Male, J2 Screw_Terminal_01x04, Q1 2N7002E, Q10 IRLB8721PBF, Q11 IRLB8721PBF, Q2 DMN65D8L-7, Q3 DMN65D8L-7, Q5 IRF4905, Q6 IRLB8721PBF, Q7 IRLB8721PBF, Q8 IRLB8721PBF, Q9 IRLB8721PBF, SW1 1301.9314, SW2 D6C50 F1 LFS, SW3 D6C40 F1 LFS, U1 ATmega328P-PU, U10 IRS2004, U3 uA7810, U4 LM7805_TO220, U6 LM339, U7 MCP601-xP, U8 IRS2004, U9 IRS2004, Y1 9B-16.000MBBK-B

Commit message: Ready for new Digikey BOM
Parts:
- removed C15, C9: 22uF, Capacitor_SMD:C_0805_2012Metric_Pad1.15x1.40mm_HandSolder, symbol Device:C
- removed C34, C35, C36: 0.47uF, Capacitor_SMD:C_0805_2012Metric_Pad1.15x1.40mm_HandSolder, symbol Device:C
- removed Q1: 2N7002E, Package_TO_SOT_SMD:SOT-23, symbol Transistor_FET:2N7002E
- removed R21, R24: 1, Resistor_THT:Power_Resistor_TH, symbol Device:R_US
- removed R4: 10K, Resistor_SMD:R_0805_2012Metric_Pad1.15x1.40mm_HandSolder, symbol Device:R_US
- removed R9: 1K, Resistor_SMD:R_0805_2012Metric_Pad1.15x1.40mm_HandSolder, symbol Device:R_US
- removed RV1: 5K, Potentiometer_SMD:Trimmer_Pot_SM, symbol Device:R_POT
- removed SW1: 1301.9314, Button_Switch_SMD:Tactile_Switch_SM, symbol Switch:SW_Push
- added C? (x2): 47uF, Capacitor_THT:CP_Radial_D10.0mm_P5.00mm, symbol Device:CP
- added C? (x4): 1uF, Capacitor_SMD:C_0805_2012Metric_Pad1.15x1.40mm_HandSolder, symbol Device:C
- added C?: 0.1uF, Capacitor_SMD:C_0805_2012Metric_Pad1.15x1.40mm_HandSolder, symbol Device:C
- added C? (x2): 1uF, Capacitor_SMD:C_0805_2012Metric_Pad1.15x1.40mm_HandSolder, symbol Device:C_Small
- added D?: BAT54HT1G, Diode_SMD:D_SOD-323_HandSoldering, symbol Diode:1N914
- added J? (x7): Conn_01x02_Female, symbol Connector:Conn_01x02_Female
- added J? (x2): Conn_01x03_Male, symbol Connector:Conn_01x03_Male
- added JP?: SolderJumper_2_Open, Jumper:Solder_Jumper_2_Pin_5A, symbol Jumper:SolderJumper_2_Open
- added Q?: DMN65D8L-7, Package_TO_SOT_SMD:SOT-23, symbol Transistor_FET:DMN67D7L
- added R?: 5K, Resistor_SMD:R_0805_2012Metric_Pad1.15x1.40mm_HandSolder, symbol Device:R_US
- added R? (x2): 10K, Resistor_SMD:R_0805_2012Metric_Pad1.15x1.40mm_HandSolder, symbol Device:R_US
- added R? (x2): 100K, Resistor_SMD:R_0805_2012Metric_Pad1.15x1.40mm_HandSolder, symbol Device:R_US
- added SW?: SW_Push_DPDT, symbol Switch:SW_Push_DPDT
- added SW?: 1301.9314, Button_Switch_SMD:Tactile_Switch_SM, symbol Switch:SW_Push
- added SW?: 1301.9314, Button_Switch_THT:Pushbutton_Switch_TH, symbol Switch:SW_Push
- added TP? (x7): TestPoint, TestPoint:TestPoint_THTPad_1.0x1.0mm_Drill0.5mm, symbol Connector:TestPoint
- C1, C2: value 10uF -> 1uF
- C21, C28, C29, C30: value 0.1uF -> 1uF
- R11, R12: value 10K -> 100K
- R22: value 40K -> 50K
- R25: Power (none) -> 1W
- R29, R30: value 1 -> 0.47; Power (none) -> 3W
- R49, R50, R51: value 1K -> 100K
- R6, R7: value 220 -> 10K
Connections:
- net labels added: BTN_nRST, EXT_nRST, I_ERR, I_FILT, I_THRESH, V_MOTOR, nI_TRIG
- net labels removed: Vdrive, nI_ERR
- wire segments 271 -> 335
- no-connect marks 4 -> 5
Other:
- note added: "AUX"
- note added: "CURRENT SENSE"
- note added: "LED Output"
- note added: "START"
- note added: "User Input"
- note removed: "Latching Circuit\n"
- note removed: "OVERCURRENT"
- moved on the sheet: C1, C10, C11, C13, C14, C17, C2, C20, C21, C23, C24, C25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

Commit message: Updated Some Passives
Parts:
- removed C31: 1nF, Capacitor_SMD:C_0805_2012Metric_Pad1.15x1.40mm_HandSolder, symbol Device:C_Small
- removed C32: 100pF, Capacitor_SMD:C_0805_2012Metric_Pad1.15x1.40mm_HandSolder, symbol Device:C_Small
- C27: value 10nF -> 15nF
- R26, R27, R28: value 4.7 -> 10
- R?: value 5K -> 10K
Connections:
- wire segments 335 -> 329
Other:
- moved on the sheet: C27, D1, D2, D3, D4, D5, D6, D9, J?, Q2, Q3, Q?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

Commit message: Removed DPDT Switch
Parts:
- removed SW?: SW_Push_DPDT, symbol Switch:SW_Push_DPDT
- gave numbers to parts that had none: 39
Connections:
- net labels removed: BTN_nRST, EXT_nRST
- wire segments 329 -> 326
- no-connect marks 5 -> 2

Commit message: Reannotated Schematic and Filtered BEMF
Parts:
- added J6, J7, J8: Conn_01x02_Female, symbol Connector:Conn_01x02_Female
- renumbered C4 to C1, C8 to C10, C17 to C11, C5 to C12, C6 to C13, C20 to C14, C18 to C15, C19 to C16, C13 to C17, C14 to C18, C16 to C19, C9 to C2, C22 to C20, C10 to C21, C31 to C22, C37 to C23, C21 to C24, C23 to C25, C24 to C26, C25 to C27, C26 to C28, C27 to C29, C12 to C3, C28 to C30, C29 to C31, C30 to C32, C32 to C33, C33 to C36, C3 to C4, C15 to C5, C7 to C6, C11 to C7, C1 to C8, C2 to C9, D3 to D1, D13 to D10, D10 to D11, D11 to D12, D7 to D13, D1 to D3, D9 to D7, D12 to D8, D8 to D9, J7 to J10, J8 to J11, J9 to J12, J10 to J13, J11 to J14, J6 to J9, R3 to R1, R11 to R10, R12 to R11, R14 to R12, R4 to R13, R9 to R14, R19 to R16, R21 to R17, R17 to R18, R16 to R19, R18 to R20, R20 to R21, R26 to R24, R27 to R25, R28 to R26, R25 to R27, R29 to R28, R24 to R29, R1 to R3, R31 to R30, R35 to R31, R39 to R32, R30 to R33, R32 to R34, R33 to R35, R34 to R36, R36 to R37, R37 to R38, R38 to R39, R5 to R4, R46 to R43, R47 to R44, R48 to R45, R43 to R46, R44 to R47, R45 to R48, R8 to R5, R10 to R6, R13 to R7, R6 to R8, R7 to R9, SW2 to SW1, SW3 to SW2, SW4 to SW3, SW5 to SW4, TP19 to TP1, TP17 to TP10, TP3 to TP11, TP29 to TP12, TP12 to TP13, TP2 to TP14, TP28 to TP15, TP18 to TP16, TP5 to TP17, TP4 to TP18, TP30 to TP19, TP25 to TP2, TP31 to TP20, TP1 to TP21, TP6 to TP22, TP7 to TP23, TP8 to TP24, TP9 to TP25, TP10 to TP26, TP11 to TP27, TP32 to TP28, TP33 to TP29, TP20 to TP3, TP34 to TP30, TP13 to TP31, TP14 to TP32, TP15 to TP33, TP35 to TP34, TP36 to TP35, TP37 to TP36, TP16 to TP37, TP21 to TP4, TP22 to TP5, TP26 to TP6, TP27 to TP7, TP23 to TP8, TP24 to TP9, U3 to U2, U4 to U3, U6 to U4, U7 to U5, U8 to U6, U9 to U7, U10 to U8
Connections:
- wire segments 326 -> 332
Other:
- moved on the sheet: J5, R19, TP14, TP18, TP19, U4A

Commit message: Reannotated and Cleaned Up Schematic
Parts:
- removed C20, C8, C9: 1uF, Capacitor_SMD:C_0805_2012Metric_Pad1.15x1.40mm_HandSolder, symbol Device:C_Small
- removed C26, C27: 0.1uF, Capacitor_SMD:C_0805_2012Metric_Pad1.15x1.40mm_HandSolder, symbol Device:C
- removed D2, D5: LTST-C171KRKT, LED_SMD:LED_0805_2012Metric_Pad1.15x1.40mm_HandSolder, symbol Device:LED
- removed R14, R15, R37, R40: 100K, Resistor_SMD:R_0805_2012Metric_Pad1.15x1.40mm_HandSolder, symbol Device:R_US
- removed R17, R8: 10K, Resistor_SMD:R_0805_2012Metric_Pad1.15x1.40mm_HandSolder, symbol Device:R_US
- removed R25, R31, R41: 10, Resistor_SMD:R_0805_2012Metric_Pad1.15x1.40mm_HandSolder, symbol Device:R_US
- removed TP12, TP13: TestPoint, TestPoint:TestPoint_Keystone_5000-5004_Miniature, symbol Connector:TestPoint
- removed TP20, TP21, TP25, TP29, TP35, TP6, TP7: TestPoint, TestPoint:TestPoint_THTPad_1.0x1.0mm_Drill0.5mm, symbol Connector:TestPoint
- removed TP39: PHASE_B, TestPoint:TestPoint_Keystone_5000-5004_Miniature, symbol Connector:TestPoint
- removed TP40: PHASE_C, TestPoint:TestPoint_Keystone_5000-5004_Miniature, symbol Connector:TestPoint
- added C13, C14, C24: 1uF, Capacitor_SMD:C_0805_2012Metric_Pad1.15x1.40mm_HandSolder, symbol Device:C_Small
- added C28, C29: 0.1uF, Capacitor_SMD:C_0805_2012Metric_Pad1.15x1.40mm_HandSolder, symbol Device:C
- added D10: LTST-C171TBKT, LED_SMD:LED_0805_2012Metric_Pad1.15x1.40mm_HandSolder, symbol Device:LED
- added D9: LTST-C171GKT, LED_SMD:LED_0805_2012Metric_Pad1.15x1.40mm_HandSolder, symbol Device:LED
- added J15: Conn_01x04_Male, symbol Connector:Conn_01x04_Male
- added R12, R20, R22, R43, R44, R45: 100K, Resistor_SMD:R_0805_2012Metric_Pad1.15x1.40mm_HandSolder, symbol Device:R_US
- added R33, R35, R36: 10, Resistor_SMD:R_0805_2012Metric_Pad1.15x1.40mm_HandSolder, symbol Device:R_US
- added TP1, TP3, TP31, TP32, TP33, TP4, TP5, TP8, TP9: TestPoint, TestPoint:TestPoint_THTPad_1.0x1.0mm_Drill0.5mm, symbol Connector:TestPoint
- C25: renamed from C24; value 1uF -> 0.1uF
- D3: value LTST-C171GKT -> LTST-C171KRKT; Color Green -> Red
- D6: value LTST-C171GKT -> LTST-C171KRKT
- D7: value LTST-C171TBKT -> LTST-C171GKT; Color Blue -> Green
- J4: renamed from J2; value Screw_Terminal_01x04 -> Screw_Terminal
- R10: value 100K -> 10K
- R26: value 10 -> 10K
- R39: value 100K -> 10
- R4: value 800 -> 300
- R5: value 300 -> 800
- TP10, TP16: footprint TestPoint:TestPoint_Keystone_5000-5004_Miniature -> TestPoint:TestPoint_THTPad_1.0x1.0mm_Drill0.5mm
- TP38: value PHASE_A -> TestPoint; footprint TestPoint:TestPoint_Keystone_5000-5004_Miniature -> TestPoint:TestPoint_THTPad_1.0x1.0mm_Drill0.5mm
- renumbered C12 to C10, C13 to C11, C14 to C12, C21 to C20, C23 to C21, C28 to C23, C29 to C26, C25 to C27, C10 to C8, C11 to C9, D8 to D2, D9 to D5, D10 to D8, J3 to J2, J4 to J3, R16 to R14, R22 to R15, R23 to R16, R19 to R17, R20 to R19, R27 to R21, R28 to R23, R21 to R24, R33 to R25, R29 to R27, R43 to R28, R44 to R29, R45 to R30, R24 to R31, R35 to R34, R30 to R37, R34 to R40, R36 to R41, R49 to R46, R50 to R47, R51 to R48, R46 to R49, R47 to R50, R48 to R51, R12 to R8, TP5 to TP12, TP32 to TP13, TP9 to TP20, TP33 to TP21, TP4 to TP25, TP8 to TP29, TP3 to TP35, TP1 to TP6, TP31 to TP7, U5 to U4, U4 to U5
Connections:
- net labels added: A_FILT, B_FILT, C_FILT, EFUSE_GATE, GATE_A_HI, GATE_A_LO, GATE_B_HI, GATE_B_LO, GATE_C_HI, GATE_C_LO, I2C_SCL, I2C_SDA
- wire segments 332 -> 333
- no-connect marks 2 -> 0
Other:
- note added: "Back EMF Sense"
- note added: "Connectors"
- note added: "Current Sense"
- note added: "Power & Protection"
- note added: "System Output"
- note added: "Test Points"
- note removed: "Back EMF Sensing\nCrossover Detection"
- note removed: "CURRENT SENSE"
- note removed: "Input Connections"
- note removed: "LED Output"
- note removed: "POWER"
- note removed: "Voltage Generation & Protection"
- moved on the sheet: C1, C10, C11, C12, C15, C16, C17, C18, C19, C2, C20, C21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

Commit message: Ready For Footprints
Parts:
- removed J6, J7, J8: Conn_01x02_Female, symbol Connector:Conn_01x02_Female
- added R52: 100, Resistor_SMD:R_0805_2012Metric_Pad1.15x1.40mm_HandSolder, symbol Device:R_US
- added SW5: SW_Push_DPDT, symbol Switch:SW_Push_DPDT
- R28, R29, R30: value 1K -> 10K
Connections:
- net labels added: BTN_nRST, EXT_nRST
- wire segments 333 -> 336
- no-connect marks 0 -> 3
Other:
- moved on the sheet: J5, R17, R28, R29, R30, U5A

Commit message: Ready for Parts Placement
Parts:
- C1, C19, C2, C7: footprint Capacitor_THT:CP_Radial_D10.0mm_P5.00mm -> Capacitor_THT:CP_Radial_D5.0mm_P2.00mm
- J10, J11, J12, J13, J14, J5, J9: footprint (none) -> Connector_PinHeader_2.54mm:PinHeader_1x02_P2.54mm_Vertical
- J15: footprint (none) -> Connector_PinHeader_2.54mm:PinHeader_1x04_P2.54mm_Vertical
- J2, J3: footprint (none) -> Connector_PinHeader_2.54mm:PinHeader_1x03_P2.54mm_Vertical
- SW3: footprint Button_Switch_THT:Pushbutton_Switch_TH -> Button_Switch_SMD:Tactile_Switch_SM
- SW5: footprint (none) -> Button_Switch_SMD:Slide_Switch_DPDT_SMD
Other:
- moved on the sheet: C1, C10, C11, C12, C13, C14, C15, C16, C17, C18, C19, C2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

Commit message: Cleaned Up Repo
Parts:
- removed Q4: DMN65D8L-7, Package_TO_SOT_SMD:SOT-23, symbol Transistor_FET:DMN67D7L
- removed R18: 10K, Resistor_SMD:R_0805_2012Metric_Pad1.15x1.40mm_HandSolder, symbol Device:R_US
- added U9: NSL-32, symbol Isolator:NSL-32
- R14: value 1K -> 150
Connections:
- wire segments 336 -> 340
Other:
- moved on the sheet: R14, R24
Changed lines of the file:
@@
 L Device:R_US R24
 U 1 1 5E18B694
-P 9100 1500
-F 0 "R24" H 8950 1500 50  0000 C CNN
-F 1 "1K" H 8950 1400 50  0000 C CNN
-F 2 "Resistor_SMD:R_0805_2012Metric_Pad1.15x1.40mm_HandSolder" V 9140 1490 50  0001 C CNN
-F 3 "~" H 9100 1500 50  0001 C CNN
-	1    9100 1500
+P 9100 1550
+F 0 "R24" H 8950 1550 50  0000 C CNN
+F 1 "1K" H 8950 1450 50  0000 C CNN
+F 2 "Resistor_SMD:R_0805_2012Metric_Pad1.15x1.40mm_HandSolder" V 9140 1540 50  0001 C CNN
+F 3 "~" H 9100 1550 50  0001 C CNN
+	1    9100 1550
 	1    0    0    -1
 $EndComp
@@
 L Device:R_US R14
 U 1 1 5E1991B6
-P 8200 1850
-F 0 "R14" V 8000 1850 50  0000 C CNN
-F 1 "1K" V 8100 1850 50  0000 C CNN
-F 2 "Resistor_SMD:R_0805_2012Metric_Pad1.15x1.40mm_HandSolder" V 8240 1840 50  0001 C CNN
-F 3 "~" H 8200 1850 50  0001 C CNN
-	1    8200 1850
+P 8100 1850
+F 0 "R14" V 7900 1850 50  0000 C CNN
+F 1 "150" V 8000 1850 50  0000 C CNN
+F 2 "Resistor_SMD:R_0805_2012Metric_Pad1.15x1.40mm_HandSolder" V 8140 1840 50  0001 C CNN
+F 3 "~" H 8100 1850 50  0001 C CNN
+	1    8100 1850
 	0    1    1    0
 $EndComp
 Text Label 7550 1850 0    50   ~ 0
 EFUSE_EN
-$Comp
-L Device:R_US R18
-U 1 1 5E0E4EED
-P 8500 2000
-F 0 "R18" H 8350 2000 50  0000 C CNN
-F 1 "10K" H 8350 1900 50  0000 C CNN
-F 2 "Resistor_SMD:R_0805_2012Metric_Pad1.15x1.40mm_HandSolder" V 8540 1990 50  0001 C CNN
-F 3 "~" H 8500 2000 50  0001 C CNN
-	1    8500 2000
-	1    0    0    -1
-$EndComp
-$Comp
-L power:GNDD #PWR084
-U 1 1 5E62DD30
-P 9100 2150
-F 0 "#PWR084" H 9100 1900 50  0001 C CNN
-F 1 "GNDD" H 9104 1995 50  0000 C CNN
-F 2 "" H 9100 2150 50  0001 C CNN
-F 3 "" H 9100 2150 50  0001 C CNN
-	1    9100 2150
-	1    0    0    -1
-$EndComp
 Connection ~ 8600 1000
 $Comp
@@
 Wire Wire Line
 	8550 2750 9000 2750
-$Comp
-L Transistor_FET:DMN67D7L Q4
-U 1 1 5E2655F0
-P 9000 1850
-F 0 "Q4" H 9200 1900 50  0000 L CNN
-F 1 "DMN65D8L-7" H 9200 1800 50  0000 L CNN
-F 2 "Package_TO_SOT_SMD:SOT-23" H 9200 1775 50  0001 L CIN
-F 3 "http://www.diodes.com/assets/Datasheets/DMN67D7L.pdf" H 9000 1850 50  0001 L CNN
-	1    9000 1850
-	1    0    0    -1
-$EndComp
-Wire Wire Line
-	8350 1850 8500 1850
 Text Label 8150 1000 0    50   ~ 0
 V_MOTOR
@@
 	9250 1300 9250 1350
 Wire Wire Line
-	8800 1850 8500 1850
-Connection ~ 8500 1850
-Wire Wire Line
-	9100 2050 9100 2150
-$Comp
-L power:GNDD #PWR077
-U 1 1 5FBEC279
-P 8500 2150
-F 0 "#PWR077" H 8500 1900 50  0001 C CNN
-F 1 "GNDD" H 8504 1995 50  0000 C CNN
-F 2 "" H 8500 2150 50  0001 C CNN
-F 3 "" H 8500 2150 50  0001 C CNN
-	1    8500 2150
-	1    0    0    -1
-$EndComp
-Wire Wire Line
 	8000 1000 8600 1000
 $Comp
@@
 Wire Wire Line
 	8600 1350 8950 1350
-Connection ~ 9250 1350
-Connection ~ 9100 1350
-Wire Wire Line
-	9100 1350 9250 1350
 Wire Wire Line
 	8950 1300 8950 1350
-Connection ~ 8950 1350
-Wire Wire Line
-	8950 1350 9100 1350
 Wire Wire Line
 	8950 1100 8950 1000
@@
 $EndComp
 Wire Wire Line
-	7550 1850 8050 1850
+	7550 1850 7950 1850
 Wire Wire Line
 	7800 2750 8250 2750
@@
 NoConn ~ 7050 6500
 NoConn ~ 7050 6700
+$Comp
+L power:GNDPWR #PWR084
+U 1 1 5E09A255
+P 9100 2100
+F 0 "#PWR084" H 9100 1900 50  0001 C CNN
+F 1 "GNDPWR" H 9104 1946 50  0000 C CNN
+F 2 "" H 9100 2050 50  0001 C CNN
+F 3 "" H 9100 2050 50  0001 C CNN
+	1    9100 2100
+	1    0    0    -1
+$EndComp
+Wire Wire Line
+	9100 2050 9100 2100
+$Comp
+L Isolator:NSL-32 U9
+U 1 1 5E0D9513
+P 8650 1950
+F 0 "U9" H 8650 2267 50  0000 C CNN
+F 1 "NSL-32" H 8650 2176 50  0000 C CNN
+F 2 "" H 8650 1650 50  0001 C CNN
+F 3 "http://lunainc.com/wp-content/uploads/2016/06/NSL-32.pdf" H 8700 1950 50  0001 C CNN
+	1    8650 1950
+	1    0    0    -1
+$EndComp
+Wire Wire Line
+	8350 1850 8250 1850
+$Comp
+L power:GNDD #PWR077
+U 1 1 5E17C602
+P 8350 2100
+F 0 "#PWR077" H 8350 1850 50  0001 C CNN
+F 1 "GNDD" H 8354 1945 50  0000 C CNN
+F 2 "" H 8350 2100 50  0001 C CNN
+F 3 "" H 8350 2100 50  0001 C CNN
+	1    8350 2100
+	1    0    0    -1
+$EndComp
+Wire Wire Line
+	8350 2050 8350 2100
+Wire Wire Line
+	8950 2050 9100 2050
+Wire Wire Line
+	8950 1850 9100 1850
+Wire Wire Line
+	9100 1850 9100 1700
+Wire Wire Line
+	8950 1350 9100 1350
+Connection ~ 8950 1350
+Connection ~ 9250 1350
+Wire Wire Line
+	9100 1350 9100 1400
+Connection ~ 9100 1350
+Wire Wire Line
+	9100 1350 9250 1350
 $EndSCHEMATC
